Commit message: fix: configure dual VLP-16 setup (ports, sync, crop box)

File: autobus_sensor_kit_description/urdf/sensor_kit.xacro (robot description, xacro)
@@ -19,5 +19,5 @@
     <xacro:property name="calibration" value="${xacro.load_yaml('$(arg config_dir)/sensor_kit_calibration.yaml')}"/>
     <!-- lidar -->
-    <xacro:VLP-16 parent="sensor_kit_base_link" name="velodyne_top" topic="/points_raw" hz="10" samples="220" gpu="$(arg gpu)">
+    <!-- <xacro:VLP-16 parent="sensor_kit_base_link" name="velodyne_top" topic="/points_raw" hz="10" samples="220" gpu="$(arg gpu)">
       <origin
         xyz="${calibration['sensor_kit_base_link']['velodyne_top_base_link']['x']}
@@ -28,5 +28,5 @@
              ${calibration['sensor_kit_base_link']['velodyne_top_base_link']['yaw']}"
       />
-    </xacro:VLP-16>
+    </xacro:VLP-16> -->
     <!-- <xacro:VLP-16 parent="sensor_kit_base_link" name="velodyne_left" topic="/points_raw" hz="10" samples="220" gpu="$(arg gpu)">
       <origin

File: autobus_sensor_kit_description/urdf/sensors.xacro (robot description, xacro)
@@ -3,4 +3,5 @@
   <xacro:arg name="config_dir" default="$(find autobus_sensor_kit_description)/config"/>
   <xacro:property name="calibration" value="${xacro.load_yaml('$(arg config_dir)/sensors_calibration.yaml')}"/>
+  <xacro:property name="sensor_kit_calibration" value="${xacro.load_yaml('$(arg config_dir)/sensor_kit_calibration.yaml')}"/>
   <!-- sensor kit -->
   <xacro:include filename="sensor_kit.xacro"/>
@@ -16,13 +17,25 @@
   <!-- embedded sensors -->
   <xacro:include filename="$(find velodyne_description)/urdf/VLP-16.urdf.xacro"/>
-  <!-- <xacro:VLP-16 parent="base_link" name="velodyne_rear" topic="velodyne_rear/velodyne_points" hz="10" samples="220" gpu="false">
+  <!-- Top Lidar -->
+  <xacro:VLP-16 parent="sensor_kit_base_link" name="velodyne_top" topic="/points_raw" hz="10" samples="220" gpu="$(arg gpu)">
     <origin
-      xyz="${calibration['base_link']['velodyne_rear_base_link']['x']}
-           ${calibration['base_link']['velodyne_rear_base_link']['y']}
-           ${calibration['base_link']['velodyne_rear_base_link']['z']}"
-      rpy="${calibration['base_link']['velodyne_rear_base_link']['roll']}
-           ${calibration['base_link']['velodyne_rear_base_link']['pitch']}
-           ${calibration['base_link']['velodyne_rear_base_link']['yaw']}"
+      xyz="${sensor_kit_calibration['sensor_kit_base_link']['velodyne_top_base_link']['x']}
+           ${sensor_kit_calibration['sensor_kit_base_link']['velodyne_top_base_link']['y']}
+           ${sensor_kit_calibration['sensor_kit_base_link']['velodyne_top_base_link']['z']}"
+      rpy="${sensor_kit_calibration['sensor_kit_base_link']['velodyne_top_base_link']['roll']}
+           ${sensor_kit_calibration['sensor_kit_base_link']['velodyne_top_base_link']['pitch']}
+           ${sensor_kit_calibration['sensor_kit_base_link']['velodyne_top_base_link']['yaw']}"
     />
-  </xacro:VLP-16> -->
+  </xacro:VLP-16>
+  <!-- Rear Lidar -->
+  <xacro:VLP-16 parent="sensor_kit_base_link" name="velodyne_rear" topic="/points_raw" hz="10" samples="220" gpu="$(arg gpu)">
+    <origin
+      xyz="${sensor_kit_calibration['sensor_kit_base_link']['velodyne_rear_base_link']['x']}
+           ${sensor_kit_calibration['sensor_kit_base_link']['velodyne_rear_base_link']['y']}
+           ${sensor_kit_calibration['sensor_kit_base_link']['velodyne_rear_base_link']['z']}"
+      rpy="${sensor_kit_calibration['sensor_kit_base_link']['velodyne_rear_base_link']['roll']}
+           ${sensor_kit_calibration['sensor_kit_base_link']['velodyne_rear_base_link']['pitch']}
+           ${sensor_kit_calibration['sensor_kit_base_link']['velodyne_rear_base_link']['yaw']}"
+    />
+  </xacro:VLP-16>
 </robot>
